File: Schematics/SKR mini LCD board/SKR mini LCD board.sch (KiCad schematic (older format))
At the start: 8 parts, among them J1 Connector 5x2, SW1 Reset, U1 SSD1306 0.96\" OLED

Commit message: Tweaks
Backport fix led order
Fix run FYSETC AIOII
Add more display support
Use STMST32 framework 10.0.1
Parts:
- removed D1: WS2812B, LED_SMD:LED_WS2812B_PLCC4_5.0x5.0mm_P3.2mm, symbol LED:WS2812B
- added Q1: BC547, Package_TO_SOT_THT:TO-92_Inline, symbol Transistor_BJT:BC547
- added R3: 1K, Resistor_THT:R_Axial_DIN0207_L6.3mm_D2.5mm_P10.16mm_Horizontal, symbol Device:R
Other:
- note removed: "Optional"
- moved on the sheet: BZ1
Changed lines of the file:
@@
 Sheet 1 1
 Title "SKR Mini V1.1 LCD board"
-Date "2019-09-23"
-Rev "1"
+Date "2020-08-15"
+Rev "2"
 Comp "Technik Gegg"
 Comment1 ""
@@
 L Device:Buzzer BZ1
 U 1 1 5D893D6F
-P 6300 4950
-F 0 "BZ1" H 6200 4750 50  0000 L CNN
-F 1 "Buzzer" H 6200 4650 50  0000 L CNN
-F 2 "Buzzer_Beeper:Buzzer_12x9.5RM7.6" V 6275 5050 50  0001 C CNN
-F 3 "~" V 6275 5050 50  0001 C CNN
-	1    6300 4950
+P 7200 4550
+F 0 "BZ1" H 7400 4600 50  0000 L CNN
+F 1 "Buzzer" H 7400 4500 50  0000 L CNN
+F 2 "Buzzer_Beeper:Buzzer_12x9.5RM7.6" V 7175 4650 50  0001 C CNN
+F 3 "~" V 7175 4650 50  0001 C CNN
+	1    7200 4550
 	1    0    0    -1
 $EndComp
@@
 F 3 "" H 3550 2500 50  0001 C CNN
 	1    3550 2500
-	1    0    0    -1
+	0    -1   -1   0
 $EndComp
 $Comp
@@
 L power:GND #PWR0107
 U 1 1 5D89A417
-P 5950 5150
-F 0 "#PWR0107" H 5950 4900 50  0001 C CNN
-F 1 "GND" H 5955 4977 50  0000 C CNN
-F 2 "" H 5950 5150 50  0001 C CNN
-F 3 "" H 5950 5150 50  0001 C CNN
-	1    5950 5150
+P 7100 5350
+F 0 "#PWR0107" H 7100 5100 50  0001 C CNN
+F 1 "GND" H 7105 5177 50  0000 C CNN
+F 2 "" H 7100 5350 50  0001 C CNN
+F 3 "" H 7100 5350 50  0001 C CNN
+	1    7100 5350
 	1    0    0    -1
 $EndComp
@@
 	4600 1600 4600 1850
 Wire Wire Line
-	6200 5050 5950 5050
-Wire Wire Line
-	5950 5050 5950 5150
+	7100 5250 7100 5350
 $Comp
 L power:GND #PWR0108
@@
 	4300 5400 4000 5400
 Wire Wire Line
-	6150 4300 6500 4300
-Wire Wire Line
 	5650 4400 4500 4400
 Wire Wire Line
@@
 $EndComp
 Wire Wire Line
-	6500 4300 6500 5950
-Wire Wire Line
 	4000 5950 4300 5950
 Wire Wire Line
 	4300 5600 4300 5950
-Wire Wire Line
-	6150 4850 6200 4850
-Wire Wire Line
-	6150 4600 6150 4850
 $Comp
 L power:GND #PWR0109
@@
 Connection ~ 4300 5950
 Wire Wire Line
-	4300 5950 6500 5950
+	4300 5950 6250 5950
 Wire Wire Line
 	6250 3800 6250 4200
-$Comp
-L LED:WS2812B D1
-U 1 1 5D8C3DC4
-P 3550 4500
-F 0 "D1" H 3206 4454 50  0000 R CNN
-F 1 "WS2812B" H 3206 4545 50  0000 R CNN
-F 2 "LED_SMD:LED_WS2812B_PLCC4_5.0x5.0mm_P3.2mm" H 3600 4200 50  0001 L TNN
-F 3 "https://cdn-shop.adafruit.com/datasheets/WS2812B.pdf" H 3650 4125 50  0001 L TNN
-	1    3550 4500
-	-1   0    0    1
-$EndComp
-Wire Wire Line
-	3850 4500 5650 4500
-$Comp
-L power:GND #PWR0110
-U 1 1 5D8C682F
-P 3550 4200
-F 0 "#PWR0110" H 3550 3950 50  0001 C CNN
-F 1 "GND" H 3555 4027 50  0000 C CNN
-F 2 "" H 3550 4200 50  0001 C CNN
-F 3 "" H 3550 4200 50  0001 C CNN
-	1    3550 4200
-	-1   0    0    1
-$EndComp
 Wire Wire Line
 	3400 5400 3550 5400
 Connection ~ 3550 5400
 Wire Wire Line
-	3550 4800 3550 5400
-Wire Wire Line
 	3550 5400 3550 5950
-Wire Notes Line width 12
-	2950 3850 4250 3850
-Wire Notes Line width 12
-	4250 3850 4250 5000
-Wire Notes Line width 12
-	4250 5000 2950 5000
-Wire Notes Line width 12
-	2950 5000 2950 3850
-Text Notes 3050 4950 0    50   ~ 0
-Optional
+$Comp
+L power:+5V #PWR?
+U 1 1 5F377DF5
+P 7100 4300
+F 0 "#PWR?" H 7100 4150 50  0001 C CNN
+F 1 "+5V" H 7115 4473 50  0000 C CNN
+F 2 "" H 7100 4300 50  0001 C CNN
+F 3 "" H 7100 4300 50  0001 C CNN
+	1    7100 4300
+	1    0    0    -1
+$EndComp
+Wire Wire Line
+	7100 4300 7100 4450
+$Comp
+L Device:R R3
+U 1 1 5F3793FA
+P 6550 5050
+F 0 "R3" V 6550 5050 50  0000 C CNN
+F 1 "1K" V 6450 5050 50  0000 C CNN
+F 2 "Resistor_THT:R_Axial_DIN0207_L6.3mm_D2.5mm_P10.16mm_Horizontal" V 6480 5050 50  0001 C CNN
+F 3 "~" H 6550 5050 50  0001 C CNN
+	1    6550 5050
+	0    -1   -1   0
+$EndComp
+$Comp
+L Transistor_BJT:BC547 Q1
+U 1 1 5F37DDBD
+P 7000 5050
+F 0 "Q1" H 7191 5096 50  0000 L CNN
+F 1 "BC547" H 7191 5005 50  0000 L CNN
+F 2 "Package_TO_SOT_THT:TO-92_Inline" H 7200 4975 50  0001 L CIN
+F 3 "http://www.fairchildsemi.com/ds/BC/BC547.pdf" H 7000 5050 50  0001 L CNN
+	1    7000 5050
+	1    0    0    -1
+$EndComp
+Wire Wire Line
+	7100 4650 7100 4850
+Wire Wire Line
+	6700 5050 6800 5050
+Wire Wire Line
+	6150 4300 6250 4300
+Wire Wire Line
+	6250 4300 6250 5950
+Wire Wire Line
+	6150 4600 6400 4600
+Wire Wire Line
+	6400 4600 6400 5050
 $EndSCHEMATC
